File: KiCad/JoystickPCB.kicad_pcb (KiCad board)
At the start: 2 copper layers, 6 parts, among them J1 B6B-PH-SM4-TB, U1 Pico, U2 ADS1115IDGSR

Commit message: Schematic should be finished
Parts:
- removed U1: Pico, Library:MODULE_SC0915
- added C2: 10uF, Capacitor_SMD:C_0603_1608Metric, F.Cu at (228.5, 25.3)
- added C3: 10uF, Capacitor_SMD:C_0603_1608Metric, F.Cu at (228.5, 27.8)
- added C4: 0.1uF, Capacitor_SMD:C_0603_1608Metric, F.Cu at (228.5, 30.3)
- added C5: 0.1uF, Capacitor_SMD:C_0603_1608Metric, F.Cu at (228.5, 32.8)
- added J2: B4B-PH-SM4-TBT, Library:JST_B4B-PH-SM4-TBT, F.Cu at (237.4, 36.9)
- added Q1: ~, Package_TO_SOT_SMD:SOT-363_SC-70-6, F.Cu at (246.6, 35.9)
- added R3: 10k, Resistor_SMD:R_0603_1608Metric, F.Cu at (228.5, 35.3)
- added R4: 10k, Resistor_SMD:R_0603_1608Metric, F.Cu at (228.5, 37.8)
- added R5: 10k, Resistor_SMD:R_0603_1608Metric, F.Cu at (228.5, 40.3)
- added R6: 10k, Resistor_SMD:R_0603_1608Metric, F.Cu at (228.5, 42.8)
- added U3: ICM-20948, Sensor_Motion:InvenSense_QFN-24_3x3mm_P0.4mm, F.Cu at (247.0, 31.3)
- added U4: MIC5225-1.8YM5-TR, Library:SOT-23-5_M5_MCH, F.Cu at (247.0, 26.4)
- J1: value B6B-PH-SM4-TB -> B4B-PH-SM4-TBT; footprint Library:JST_B6B-PH-SM4-TB -> Library:JST_B4B-PH-SM4-TBT
- moved J1 98.5 mm to (237.4, 27.3), turned to 0 degrees
Connections:
- net /A3.3V renamed /3.3V
- J1 pad 2: /AGND -> /GND
- J1 pad 3: /A0 -> /SDA
- J1 pad 4: /A1 -> /SCL
- J1 pad SH1: (no net) -> unconnected-(J1-SHIELD-PadSH1)
- J1 pad SH2: (no net) -> unconnected-(J1-SHIELD__1-PadSH2)

Commit message: Started work on PCB design
Parts:
- moved U4 124.3 mm to (136.4, 83.0)
- moved J1 113.2 mm to (131.5, 67.0), turned to 90 degrees
- moved Q1 107.1 mm to (152.1, 86.3)
- moved U3 101.6 mm to (160.4, 84.5)
- moved R6 97.5 mm to (141.0, 86.0)
- moved R5 92.8 mm to (145.0, 81.0)
- moved C2 92.3 mm to (141.8, 57.0)
- moved C3 90.2 mm to (145.0, 62.0)
- moved R4 81.0 mm to (155.0, 72.0)
- moved C5 78.7 mm to (162.0, 75.0)
- moved R3 74.8 mm to (170.0, 82.0)
- moved C4 70.3 mm to (182.0, 83.0)
- moved J2 58.1 mm to (186.5, 65.0), turned to -90 degrees
- moved U2 30.4 mm to (170.0, 68.0), turned to 180 degrees
- moved R1 29.2 mm to (166.0, 54.0)
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Connections:
- C1 pad 2: /AGND -> /GND
- C2 pad 1: Net-(U4-EN) -> /3.3V
- J2 pad 2: /GND -> /A1
- J2 pad 4: /A1 -> /GND
- U2 pad 3: /AGND -> /GND
- U4 pad 1: Net-(U4-EN) -> /3.3V
- U4 pad 3: Net-(U4-EN) -> /3.3V
Routing:
- net /GND: track 0.00 -> 22.6 mm
- net /A1: track 0.00 -> 13.4 mm
- net /A0: track 0.00 -> 12.8 mm
Other:
- board outline added: 68 x 53 mm
- board text added: "Joystick"
- board text added: "Microcontroller"

Commit message: Continued work on PCB layout
Parts:
- moved C4 28.3 mm to (155.3, 73.7)
- moved R6 25.5 mm to (147.9, 61.5)
- moved Q1 24.5 mm to (142.2, 63.9)
- moved R3 22.8 mm to (148.4, 74.7)
- moved R5 20.9 mm to (152.4, 61.5)
- moved U3 18.6 mm to (156.8, 66.3)
- moved U4 17.1 mm to (145.5, 68.5)
- moved C2 15.2 mm to (140.8, 72.2)
- moved R4 10.7 mm to (157.0, 61.5), turned to 180 degrees
- moved C3 8.15 mm to (150.4, 68.1)
- moved R1 7.63 mm to (167.8, 61.4)
- moved R2 7.63 mm to (172.3, 61.4)
- moved J2 3.97 mm to (182.6, 65.7)
- moved C5 3.22 mm to (159.1, 73.7), turned to 180 degrees
Routing:
- net /3.3V: track 0.00 -> 38.4 mm
- net /1.8V: track 0.00 -> 23.4 mm, vias 0 -> 2
- net /GND: track 22.6 -> 44.4 mm, vias 0 -> 2
- net /SDA: track 0.00 -> 13.2 mm
- net /A0: track 12.8 -> 0.00 mm
- net /A1: track 13.4 -> 2.25 mm
- net /SCL: track 0.00 -> 9.18 mm
- net Net-(U3-REGOUT): track 0.00 -> 8.74 mm, vias 0 -> 2

Commit message: Finished initial PCB design
Parts:
- added REF**: MountingHole_3.2mm_M3_DIN965_Pad, MountingHole:MountingHole_3.2mm_M3_DIN965_Pad, F.Cu at (130.0, 77.0)
- added REF**: MountingHole_3.2mm_M3_DIN965_Pad, MountingHole:MountingHole_3.2mm_M3_DIN965_Pad, F.Cu at (184.0, 77.0)
- added REF**: MountingHole_3.2mm_M3_DIN965_Pad, MountingHole:MountingHole_3.2mm_M3_DIN965_Pad, F.Cu at (130.0, 57.0)
- added REF**: MountingHole_3.2mm_M3_DIN965_Pad, MountingHole:MountingHole_3.2mm_M3_DIN965_Pad, F.Cu at (184.0, 57.0)
- moved R3 9.70 mm to (148.0, 65.0)
- moved J2 1.32 mm to (182.2, 67.0)
Routing:
- net /3.3V: track 38.4 -> 97.1 mm, vias 0 -> 4
- net /GND: track 44.4 -> 99.2 mm, vias 2 -> 4
- net /SDA: track 13.2 -> 57.7 mm, vias 0 -> 2
- net /SCL: track 9.18 -> 52.6 mm, vias 0 -> 2
- net /1.8V: track 23.4 -> 58.0 mm
- net /SCL_1.8V: track 0.06 -> 25.2 mm, vias 0 -> 2
- net /SDA_1.8V: track 0.00 -> 16.7 mm, vias 0 -> 2
- net /A0: track 0.00 -> 8.06 mm
- net /A1: track 2.25 -> 8.26 mm
- net Net-(U3-REGOUT): track 8.74 -> 12.4 mm
Other:
- board size 68 x 53 mm -> 62 x 28 mm
- board text added: "1.0"
- board text added: "11/9/24"
- board text added: "By Robbie Leslie"
- board text added: "Joystick ADC + IMU Breakout Board"
- board text added: "Joystick physical dimentions"
