File: Joystick/KiCad/JoystickPCB.kicad_sch (KiCad schematic)
At the start: 17 parts, among them J1 B4B-PH-SM4-TBT, J2 B4B-PH-SM4-TBT, U2 ADS1115IDGSR, U3 ICM-20948, U4 MIC5225-1.8YM5-TR

Commit message: Changed I2C pullups to 4.7k
Parts:
- R1, R2, R4, R5: value 10k -> 4.7k
Changed lines of the file:
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@@
 			)
 		)
-		(property "Value" "10k"
+		(property "Value" "4.7k"
 			(at 186.69 142.2399 0)
 			(effects
@@
 			)
 		)
-		(property "Value" "10k"
+		(property "Value" "4.7k"
 			(at 156.21 64.7699 0)
 			(effects
@@
 			)
 		)
-		(property "Value" "10k"
+		(property "Value" "4.7k"
 			(at 195.58 142.2399 0)
 			(effects
@@
 			)
 		)
-		(property "Value" "10k"
+		(property "Value" "4.7k"
 			(at 156.21 30.4799 0)
 			(effects

Commit message: Removed extra I2C pullups
Parts:
- removed R3, R6: 10k, Resistor_SMD:R_0603_1608Metric, symbol Device:R
Other:
- note added: "Need to add another connector for the fingerprint reader and 1-2 more for ultrasonic sensors"
- note added: "Need to switch the microcontroller connector for 7 pin connector probably (depends on fingerprint reader)"
- note removed: "Need to add another connector for the fingerprint reader"
- note removed: "Need to switch the microcontroller connector for 7 pin connector probably"
Changed lines of the file:
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@@
 	(paper "A4")
-	(junction
-		(at 153.67 73.66)
-		(diameter 0)
-		(color 0 0 0 0)
-	)
 	(junction
 		(at 97.79 29.21)
@@
 	)
 	(junction
-		(at 153.67 41.91)
-		(diameter 0)
-		(color 0 0 0 0)
-	)
-	(junction
 		(at 224.79 77.47)
 		(diameter 0)
@@
 	(wire
 		(pts
-			(xy 153.67 73.66) (xy 154.94 73.66)
-		)
-		(stroke
-			(width 0)
-			(type default)
-		)
-	)
-	(wire
-		(pts
 			(xy 184.15 127) (xy 184.15 137.16)
 		)
@@
 	(wire
 		(pts
-			(xy 143.51 41.91) (xy 153.67 41.91)
-		)
-		(stroke
-			(width 0)
-			(type default)
-		)
-	)
-	(wire
-		(pts
 			(xy 153.67 39.37) (xy 154.94 39.37)
 		)
@@
 	(wire
 		(pts
-			(xy 153.67 41.91) (xy 154.94 41.91)
+			(xy 143.51 41.91) (xy 154.94 41.91)
 		)
 		(stroke
@@
 	(wire
 		(pts
-			(xy 153.67 87.63) (xy 153.67 95.25)
-		)
-		(stroke
-			(width 0)
-			(type default)
-		)
-	)
-	(wire
-		(pts
 			(xy 201.93 43.18) (xy 212.09 43.18)
 		)
@@
 	(wire
 		(pts
-			(xy 153.67 41.91) (xy 153.67 44.45)
-		)
-		(stroke
-			(width 0)
-			(type default)
-		)
-	)
-	(wire
-		(pts
 			(xy 237.49 55.88) (xy 248.92 55.88)
 		)
@@
 	(wire
 		(pts
-			(xy 153.67 73.66) (xy 153.67 80.01)
-		)
-		(stroke
-			(width 0)
-			(type default)
-		)
-	)
-	(wire
-		(pts
 			(xy 153.67 55.88) (xy 153.67 59.69)
 		)
@@
 	(wire
 		(pts
-			(xy 143.51 73.66) (xy 153.67 73.66)
+			(xy 143.51 73.66) (xy 154.94 73.66)
 		)
 		(stroke
@@
 		)
 	)
-	(text "Need to add another connector for the fingerprint reader"
-		(exclude_from_sim no)
-		(at 53.086 188.722 0)
+	(text "Need to add another connector for the fingerprint reader and 1-2 more for ultrasonic sensors"
+		(exclude_from_sim no)
+		(at 62.484 179.07 0)
 		(effects
 			(font
@@
 		)
 	)
-	(text "Need to switch the microcontroller connector for 7 pin connector probably "
-		(exclude_from_sim no)
-		(at 64.262 103.378 0)
+	(text "Need to switch the microcontroller connector for 7 pin connector probably (depends on fingerprint reader)"
+		(exclude_from_sim no)
+		(at 65.278 103.378 0)
 		(effects
 			(font
@@
 	(label "GND"
 		(at 224.79 81.28 0)
-		(fields_autoplaced yes)
-		(effects
-			(font
-				(size 1.27 1.27)
-			)
-			(justify left bottom)
-		)
-	)
-	(label "1.8V"
-		(at 153.67 95.25 0)
 		(fields_autoplaced yes)
 		(effects
@@
 	)
 	(symbol
-		(lib_id "Device:R")
-		(at 153.67 48.26 0)
-		(unit 1)
-		(exclude_from_sim no)
-		(in_bom yes)
-		(on_board yes)
-		(dnp no)
-		(fields_autoplaced yes)
-		(property "Reference" "R6"
-			(at 156.21 46.9899 0)
-			(effects
-				(font
-					(size 1.27 1.27)
-				)
-				(justify left)
-			)
-		)
-		(property "Value" "10k"
-			(at 156.21 49.5299 0)
-			(effects
-				(font
-					(size 1.27 1.27)
-				)
-				(justify left)
-			)
-		)
-		(property "Footprint" "Resistor_SMD:R_0603_1608Metric"
-			(at 151.892 48.26 90)
-			(effects
-				(font
-					(size 1.27 1.27)
-				)
-				(hide yes)
-			)
-		)
-		(property "Datasheet" "~"
-			(at 153.67 48.26 0)
-			(effects
-				(font
-					(size 1.27 1.27)
-				)
-				(hide yes)
-			)
-		)
-		(property "Description" "Resistor"
-			(at 153.67 48.26 0)
-			(effects
-				(font
-					(size 1.27 1.27)
-				)
-				(hide yes)
-			)
-		)
-		(pin "2"
-		)
-		(pin "1"
-		)
-		(instances
-			(project "JoystickPCB"
-				(path "/40b06a56-8aa7-465d-9cc9-72851af3998b"
-					(reference "R6")
-					(unit 1)
-				)
-			)
-		)
-	)
-	(symbol
 		(lib_id "Sensor_Motion:ICM-20948")
 		(at 224.79 50.8 0)
@@
 					(unit 1)
 				)
-			)
-		)
-	)
-	(symbol
-		(lib_id "Device:R")
-		(at 153.67 83.82 0)
-		(unit 1)
-		(exclude_from_sim no)
-		(in_bom yes)
-		(on_board yes)
-		(dnp no)
-		(fields_autoplaced yes)
-		(property "Reference" "R3"
-			(at 156.21 82.5499 0)
-			(effects
-				(font
-					(size 1.27 1.27)
-				)
-				(justify left)
-			)
-		)
-		(property "Value" "10k"
-			(at 156.21 85.0899 0)
-			(effects
-				(font
-					(size 1.27 1.27)
-				)
-				(justify left)
-			)
-		)
-		(property "Footprint" "Resistor_SMD:R_0603_1608Metric"
-			(at 151.892 83.82 90)
-			(effects
-				(font
-					(size 1.27 1.27)
-				)
-				(hide yes)
-			)
-		)
-		(property "Datasheet" "~"
-			(at 153.67 83.82 0)
-			(effects
-				(font
-					(size 1.27 1.27)
-				)
-				(hide yes)
-			)
-		)
-		(property "Description" "Resistor"
-			(at 153.67 83.82 0)
-			(effects
-				(font
-					(size 1.27 1.27)
-				)
-				(hide yes)
-			)
-		)
-		(pin "2"
-		)
-		(pin "1"
-		)
-		(instances
-			(project "JoystickPCB"
-				(path "/40b06a56-8aa7-465d-9cc9-72851af3998b"
-					(reference "R3")
-					(unit 1)
-				)

Commit message: Redesigned PCB with new connectors
Parts:
- removed J1, J2: B4B-PH-SM4-TBT, Library:JST_B4B-PH-SM4-TBT, symbol B4B-PH-SM4-TBT:B4B-PH-SM4-TBT
- added H1, H2, H3, H4: MountingHole, MountingHole:MountingHole_3.2mm_M3_DIN965_Pad_TopBottom, symbol Mechanical:MountingHole
- added J1: JST B6B-PH-SM4-TB, Connector_JST:JST_PH_B6B-PH-SM4-TB_1x06-1MP_P2.00mm_Vertical, symbol Connector_Generic:Conn_01x06
- added J2, J3: JST B4B-PH-SM4-TB, Connector_JST:JST_PH_B4B-PH-SM4-TB_1x04-1MP_P2.00mm_Vertical, symbol Connector_Generic:Conn_01x04
- added J4: JST B3B-PH-SM4-TB, Connector_JST:JST_PH_B3B-PH-SM4-TB_1x03-1MP_P2.00mm_Vertical, symbol Connector_Generic:Conn_01x03
- U1: renamed from U4; footprint SOT-23-5_M5_MCH -> Package_TO_SOT_SMD:SOT-23-5
- renumbered C2 to C1, C3 to C2, C4 to C3, C1 to C4, R4 to R1, R5 to R2, R1 to R3, R2 to R4
Connections:
- net 3.3V: now also J1.2 (Pin_2), J2.1 (Pin_1), J3.1 (Pin_1), J4.1 (Pin_1)
- net A0: now also J2.3 (Pin_3)
- net A1: now also J2.2 (Pin_2)
- net A2: now also J4.2 (Pin_2)
- net GND: now also J1.1 (Pin_1), J2.4 (Pin_4), J3.4 (Pin_4), J4.3 (Pin_3)
- net SCL: now also J1.4 (Pin_4)
- net SDA: now also J1.3 (Pin_3)
- new net RX: J1.5 (Pin_5), J3.3 (Pin_3)
- new net TX: J1.6 (Pin_6), J3.2 (Pin_2)
Other:
- note added: "Need to switch the microcontroller connector for 7 pin connector probably"
- note added: "To Fingerprint Sensor"
- note added: "To Ultrasonic Sensor"
- note removed: "Might want to swap these for right angle connectors"
- note removed: "Need to add another connector for the fingerprint reader and 1-2 more for ultrasonic sensors"
- note removed: "Need to switch the microcontroller connector for 7 pin connector probably (depends on fingerprint reader)"

Commit message: Removed I2C pullups since they will go on the main board
Parts:
- removed R3, R4: 4.7k, Resistor_SMD:R_0603_1608Metric, symbol Device:R
Changed lines of the file:
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@@
-	)
-	(junction
-		(at 184.15 127)
-		(diameter 0)
-		(color 0 0 0 0)
 	)
 	(junction
@@
 	)
 	(junction
-		(at 193.04 132.08)
-		(diameter 0)
-		(color 0 0 0 0)
-	)
-	(junction
 		(at 224.79 77.47)
 		(diameter 0)
@@
 	(wire
 		(pts
-			(xy 184.15 127) (xy 184.15 137.16)
-		)
-		(stroke
-			(width 0)
-			(type default)
-		)
-	)
-	(wire
-		(pts
 			(xy 201.93 48.26) (xy 212.09 48.26)
 		)
@@
 	(wire
 		(pts
-			(xy 193.04 144.78) (xy 193.04 156.21)
-		)
-		(stroke
-			(width 0)
-			(type default)
-		)
-	)
-	(wire
-		(pts
 			(xy 110.49 20.32) (xy 110.49 29.21)
 		)
@@
 	(wire
 		(pts
-			(xy 204.47 127) (xy 184.15 127)
-		)
-		(stroke
-			(width 0)
-			(type default)
-		)
-	)
-	(wire
-		(pts
 			(xy 227.33 20.32) (xy 227.33 29.21)
 		)
@@
 	(wire
 		(pts
-			(xy 184.15 144.78) (xy 184.15 156.21)
-		)
-		(stroke
-			(width 0)
-			(type default)
-		)
-	)
-	(wire
-		(pts
 			(xy 201.93 45.72) (xy 212.09 45.72)
 		)
@@
 	(wire
 		(pts
-			(xy 179.07 127) (xy 184.15 127)
+			(xy 179.07 127) (xy 204.47 127)
 		)
 		(stroke
@@
 	(wire
 		(pts
-			(xy 193.04 132.08) (xy 193.04 137.16)
-		)
-		(stroke
-			(width 0)
-			(type default)
-		)
-	)
-	(wire
-		(pts
 			(xy 85.09 171.45) (xy 92.71 171.45)
 		)
@@
 	(wire
 		(pts
-			(xy 189.23 132.08) (xy 193.04 132.08)
-		)
-		(stroke
-			(width 0)
-			(type default)
-		)
-	)
-	(wire
-		(pts
 			(xy 24.13 39.37) (xy 24.13 44.45)
 		)
@@
 	(wire
 		(pts
-			(xy 204.47 132.08) (xy 193.04 132.08)
+			(xy 189.23 132.08) (xy 204.47 132.08)
 		)
 		(stroke
@@
 		)
 	)
-	(label "3.3V"
-		(at 184.15 156.21 0)
-		(fields_autoplaced yes)
-		(effects
-			(font
-				(size 1.27 1.27)
-			)
-			(justify left bottom)
-		)
-	)
 	(label "GND"
 		(at 110.49 41.91 0)
@@
 	(label "3.3V"
 		(at 85.09 168.91 0)
-		(fields_autoplaced yes)
-		(effects
-			(font
-				(size 1.27 1.27)
-			)
-			(justify left bottom)
-		)
-	)
-	(label "3.3V"
-		(at 193.04 156.21 0)
 		(fields_autoplaced yes)
 		(effects
@@
 	)
 	(symbol
-		(lib_id "Device:R")
-		(at 184.15 140.97 0)
-		(unit 1)
-		(exclude_from_sim no)
-		(in_bom yes)
-		(on_board yes)
-		(dnp no)
-		(fields_autoplaced yes)
-		(property "Reference" "R3"
-			(at 186.69 139.6999 0)
-			(effects
-				(font
-					(size 1.27 1.27)
-				)
-				(justify left)
-			)
-		)
-		(property "Value" "4.7k"
-			(at 186.69 142.2399 0)
-			(effects
-				(font
-					(size 1.27 1.27)
-				)
-				(justify left)
-			)
-		)
-		(property "Footprint" "Resistor_SMD:R_0603_1608Metric"
-			(at 182.372 140.97 90)
-			(effects
-				(font
-					(size 1.27 1.27)
-				)
-				(hide yes)
-			)
-		)
-		(property "Datasheet" "~"
-			(at 184.15 140.97 0)
-			(effects
-				(font
-					(size 1.27 1.27)
-				)
-				(hide yes)
-			)
-		)
-		(property "Description" "Resistor"
-			(at 184.15 140.97 0)
-			(effects
-				(font
-					(size 1.27 1.27)
-				)
-				(hide yes)
-			)
-		)
-		(pin "2"
-		)
-		(pin "1"
-		)
-		(instances
-			(project "JoystickPCB"
-				(path "/40b06a56-8aa7-465d-9cc9-72851af3998b"
-					(reference "R3")
-					(unit 1)
-				)
-			)
-		)
-	)
-	(symbol
 		(lib_id "Device:C")
 		(at 248.92 68.58 0)
@@
 					(unit 1)
 				)
-			)
-		)
-	)
-	(symbol
-		(lib_id "Device:R")
-		(at 193.04 140.97 0)
-		(unit 1)
-		(exclude_from_sim no)
-		(in_bom yes)
-		(on_board yes)
-		(dnp no)
-		(fields_autoplaced yes)
-		(property "Reference" "R4"
-			(at 195.58 139.6999 0)
-			(effects
-				(font
-					(size 1.27 1.27)
-				)
-				(justify left)
-			)
-		)
-		(property "Value" "4.7k"
-			(at 195.58 142.2399 0)
-			(effects
-				(font
-					(size 1.27 1.27)
-				)
-				(justify left)
-			)
-		)
-		(property "Footprint" "Resistor_SMD:R_0603_1608Metric"
-			(at 191.262 140.97 90)
-			(effects
-				(font
-					(size 1.27 1.27)
-				)
-				(hide yes)
-			)
-		)
-		(property "Datasheet" "~"
-			(at 193.04 140.97 0)
-			(effects
-				(font
-					(size 1.27 1.27)
-				)
-				(hide yes)
-			)
-		)
-		(property "Description" "Resistor"
-			(at 193.04 140.97 0)
-			(effects
-				(font
-					(size 1.27 1.27)
-				)
-				(hide yes)
-			)
-		)
-		(pin "2"
-		)
-		(pin "1"
-		)
-		(instances
-			(project ""
-				(path "/40b06a56-8aa7-465d-9cc9-72851af3998b"
-					(reference "R4")
-					(unit 1)
-				)

Commit message: Switch 10uF cap sizes
Parts:
- C1, C2, C4: footprint Capacitor_SMD:C_0603_1608Metric -> Capacitor_SMD:C_0805_2012Metric
Changed lines of the file:
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@@
 			)
 		)
-		(property "Footprint" "Capacitor_SMD:C_0603_1608Metric"
+		(property "Footprint" "Capacitor_SMD:C_0805_2012Metric"
 			(at 247.3452 118.11 0)
 			(effects
@@
 			)
 		)
-		(property "Footprint" "Capacitor_SMD:C_0603_1608Metric"
+		(property "Footprint" "Capacitor_SMD:C_0805_2012Metric"
 			(at 98.7552 36.83 0)
 			(effects
@@
 			)
 		)
-		(property "Footprint" "Capacitor_SMD:C_0603_1608Metric"
+		(property "Footprint" "Capacitor_SMD:C_0805_2012Metric"
 			(at 25.0952 39.37 0)
 			(effects
