File: PIR_Ultrasonic/PIR_Ultrasonic.kicad_pcb (KiCad board)
At the start: 2 copper layers, 73.5 x 54.5 mm, 9 parts, among them J1 Conn_01x03, J2 JST B4B-PH-SM4-TB, U1 EKMC1605113

Commit message: Added comments
Other:
- board text added: "I would consider moving the PIR sensor to the other side so that the connectors are on one side and the sensor is on the other. I know we can solder it either way, but I would be specific in the design. I might also rotate the sensor 90 degrees, unless we are mounting it vertically"
- board text added: "I would personally rotate this connector 180 as well, but that is a style choice"
- board text added: "It is missing the serial number and assembly number silkscreens on the front, and the board number and revision on the back - Robbie"
- board text added: "The entire thing needs a ground fill, at least on one layer"
- board text added: "This connector needs to be rotated 180. I added the 3D model for it to make it more obvious"
- board text added: "This mounting whole is ever so slightly mis-aligned"
Changed lines of the file:
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@@
+			)
+		)
+		(model "${KIPRJMOD}/Library/3D Models/S3B-PH-SM4-TB.step"
+			(offset
+				(xyz 0 -4.5 0)
+			)
+			(scale
+				(xyz 1 1 1)
+			)
+			(rotate
+				(xyz -90 0 0)
 			)
 		)
@@
 			(rotate
 				(xyz 0 0 0)
+			)
+		)
+		(model "${KIPRJMOD}/Library/3D Models/B4B-PH-SM4-TB.step"
+			(offset
+				(xyz 0 1.8 0)
+			)
+			(scale
+				(xyz 1 1 1)
+			)
+			(rotate
+				(xyz -90 0 0)
 			)
 		)
@@
 		)
 	)
+	(gr_text "I would consider moving the PIR sensor to the other side so that the connectors are on one side and the sensor is on the other.\nI know we can solder it either way, but I would be specific in the design.\nI might also rotate the sensor 90 degrees, unless we are mounting it vertically"
+		(at 171 123.5 0)
+		(layer "Cmts.User")
+		(effects
+			(font
+				(size 1 1)
+				(thickness 0.15)
+			)
+			(justify left bottom)
+		)
+	)
+	(gr_text "This connector needs to be rotated 180.\nI added the 3D model for it to make \nit more obvious"
+		(at 108.75 121.75 0)
+		(layer "Cmts.User")
+		(effects
+			(font
+				(size 1.5 1.5)
+				(thickness 0.3)
+				(bold yes)
+			)
+			(justify left bottom)
+		)
+	)
+	(gr_text "I would personally rotate this connector 180 as well,\nbut that is a style choice"
+		(at 194 105.25 0)
+		(layer "Cmts.User")
+		(effects
+			(font
+				(size 1 1)
+				(thickness 0.15)
+			)
+			(justify left bottom)
+		)
+	)
+	(gr_text "It is missing the serial number and assembly number silkscreens on the front,\nand the board number and revision on the back - Robbie"
+		(at 126.25 143.75 0)
+		(layer "Cmts.User")
+		(effects
+			(font
+				(size 1.5 1.5)
+				(thickness 0.3)
+				(bold yes)
+			)
+			(justify left bottom)
+		)
+	)
+	(gr_text "This mounting whole is ever so slightly mis-aligned"
+		(at 136.25 69.5 0)
+		(layer "Cmts.User")
+		(effects
+			(font
+				(size 1.5 1.5)
+				(thickness 0.3)
+				(bold yes)
+			)
+			(justify left bottom)
+		)
+	)
+	(gr_text "The entire thing needs a ground fill, at least on one layer"
+		(at 201 99.5 0)
+		(layer "Cmts.User")
+		(effects
+			(font
+				(size 1 1)
+				(thickness 0.15)
+			)
+			(justify left bottom)
+		)
+	)
+	(dimension
+		(type aligned)
+		(layer "Cmts.User")
+		(pts
+			(xy 133 131.5) (xy 193 131.5)
+		)
+		(height 24.5)
+		(gr_text "60.0000 mm"
+			(at 163 154.85 0)
+			(layer "Cmts.User")
+			(effects
+				(font
+					(size 1 1)
+					(thickness 0.15)
+				)
+			)
+		)
+		(format
+			(prefix "")
+			(suffix "")
+			(units 3)
+			(units_format 1)
+			(precision 4)
+		)
+		(style
+			(thickness 0.1)
+			(arrow_length 1.27)
+			(text_position_mode 0)
+			(extension_height 0.58642)
+			(extension_offset 0.5) keep_text_aligned)
+	)
+	(dimension
+		(type aligned)
+		(layer "Cmts.User")
+		(pts
+			(xy 133 131.5) (xy 133 89.5)
+		)
+		(height -25)
+		(gr_text "42.0000 mm"
+			(at 106.85 110.5 90)
+			(layer "Cmts.User")
+			(effects
+				(font
+					(size 1 1)
+					(thickness 0.15)
+				)
+			)
+		)
+		(format
+			(prefix "")
+			(suffix "")
+			(units 3)
+			(units_format 1)
+			(precision 4)
+		)
+		(style
+			(thickness 0.1)
+			(arrow_length 1.27)
+			(text_position_mode 0)
+			(extension_height 0.58642)
+			(extension_offset 0.5) keep_text_aligned)
+	)
+	(dimension
+		(type aligned)
+		(layer "Cmts.User")
+		(pts
+			(xy 133 89.5) (xy 193 90)
+		)
+		(height -15.030501)
+		(gr_text "60.0021 mm"
+			(at 163.140249 72.920083 359.5225462)
+			(layer "Cmts.User")
+			(effects
+				(font
+					(size 1.5 1.5)
+					(thickness 0.3)
+				)
+			)
+		)
+		(format
+			(prefix "")
+			(suffix "")
+			(units 3)
+			(units_format 1)
+			(precision 4)
+		)
+		(style
+			(thickness 0.2)
+			(arrow_length 1.27)
+			(text_position_mode 0)
+			(extension_height 0.58642)
+			(extension_offset 0.5) keep_text_aligned)
+	)
+	(dimension
+		(type aligned)
+		(layer "Cmts.User")
+		(pts
+			(xy 193 90) (xy 193 131.5)
+		)
+		(height -14.25)
+		(gr_text "41.5000 mm"
+			(at 206.1 110.75 90)
+			(layer "Cmts.User")
+			(effects
+				(font
+					(size 1 1)
+					(thickness 0.15)
+				)
+			)
+		)
+		(format
+			(prefix "")
+			(suffix "")
+			(units 3)
+			(units_format 1)
+			(precision 4)
+		)
+		(style
+			(thickness 0.1)
+			(arrow_length 1.27)
+			(text_position_mode 0)
+			(extension_height 0.58642)
+			(extension_offset 0.5) keep_text_aligned)
+	)
 	(segment

Commit message: Robbie's comments resolved
Parts:
- U1: moved to B.Cu
- moved U1 6.42 mm to (169.0, 108.5), turned to 0 degrees
- moved J1 2.06 mm to (142.5, 108.5), turned to -90 degrees
- moved J2 0.71 mm to (188.5, 110.0), turned to -90 degrees
- moved H2 0.50 mm to (193.0, 89.5)
Routing:
- net /3.3V: track 123.6 -> 43.7 mm
- net /UltAnalog: track 89.7 -> 43.3 mm
- net /GND: track 53.4 -> 46.0 mm, vias 0 -> 2
- net /PIRout: track 31.3 -> 26.4 mm
- added copper zone on B.Cu, net /GND
- added copper zone on F.Cu, net /GND
Other:
- board text added: "Board Part Number: 3- Rev v1.0"
- board text added: "Serial Number: Assembly Number:"
- board text removed: "I would consider moving the PIR sensor to the other side so that the connectors are on one side and the sensor is on the other. I know we can solder it either way, but I would be specific in the design. I might also rotate the sensor 90 degrees, unless we are mounting it vertically"
- board text removed: "I would personally rotate this connector 180 as well, but that is a style choice"
- board text removed: "It is missing the serial number and assembly number silkscreens on the front, and the board number and revision on the back - Robbie"
- board text removed: "The entire thing needs a ground fill, at least on one layer"
- board text removed: "This connector needs to be rotated 180. I added the 3D model for it to make it more obvious"
- board text removed: "This mounting whole is ever so slightly mis-aligned"

Commit message: Feb 12 changes from Prof Wey's comments
Parts:
- J1: footprint Connector_JST:JST_PH_S3B-PH-SM4-TB_1x03-1MP_P2.00mm_Horizontal -> Connector_JST:JST_PH_B3B-PH-SM4-TB_1x03-1MP_P2.00mm_Vertical
- turned J1 to 90 degrees
Routing:
- net /GND: track 46.0 -> 0.00 mm
- net /UltAnalog: track 43.3 -> 79.5 mm
- net /3.3V: track 43.7 -> 46.9 mm
