File: PIR_Ultrasonic/PIR_Ultrasonic.kicad_sch (KiCad schematic)
At the start: 7 parts, among them J1 Conn_01x03, J2 JST B4B-PH-SM4-TB, U1 EKMC1605113

Commit message: Feb 12 changes from Prof Wey's comments
Parts:
- J1: footprint Connector_JST:JST_PH_S3B-PH-SM4-TB_1x03-1MP_P2.00mm_Horizontal -> Connector_JST:JST_PH_B3B-PH-SM4-TB_1x03-1MP_P2.00mm_Vertical; Manufacturer Part Number (none) -> B3B-PH-SM4-TB
- U1: Manufacturer Part Number (none) -> EKMC1605113
